Commit message: Give bottom camera more realistic angle

File: src/competition3/urdf/bottom_camera.urdf.xacro (robot description, xacro)
@@ -7,5 +7,5 @@
   <xacro:property name="cam_z" value="0.15"/>
   <xacro:property name="cam_rx" value="0.0"/>
-  <xacro:property name="cam_ry" value="0.2617994"/>
+  <xacro:property name="cam_ry" value="0.7"/>
   <xacro:property name="cam_rz" value="0.0"/>
   <xacro:macro name="bottom_camera" params="parent">
